File: electronics/cube-batteryboard/cube-batteryboard.kicad_sch (KiCad schematic)
At the start: 8 parts, among them J1 Conn_01x02, J2 Conn_01x02, SW1 SW_DPST, SW2 SW_DPST

Commit message: Fix unconnected GND circuit for J2 (pin 1)
Connections:
- net GND: now also J2.1 (Pin_1)
Changed lines of the file:
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@@
 (kicad_sch (version 20230121) (generator eeschema)
   (paper "A4")
-  (junction (at 43.18 52.07) (diameter 0) (color 0 0 0 0)
-  )
   (junction (at 43.18 34.29) (diameter 0) (color 0 0 0 0)
   )
@@
   )
   (junction (at 58.42 49.53) (diameter 0) (color 0 0 0 0)
+  )
+  (junction (at 43.18 52.07) (diameter 0) (color 0 0 0 0)
   )
   (junction (at 58.42 44.45) (diameter 0) (color 0 0 0 0)
@@
     (stroke (width 0) (type default))
   )
-  (wire (pts (xy 53.34 52.07) (xy 60.96 52.07))
-    (stroke (width 0) (type default))
-  )
   (wire (pts (xy 40.64 49.53) (xy 43.18 49.53))
     (stroke (width 0) (type default))
@@
   )
   (wire (pts (xy 45.72 44.45) (xy 43.18 44.45))
+    (stroke (width 0) (type default))
+  )
+  (wire (pts (xy 43.18 52.07) (xy 60.96 52.07))
     (stroke (width 0) (type default))
   )
@@
     (stroke (width 0) (type default))
   )
-  (wire (pts (xy 43.18 52.07) (xy 48.26 52.07))
-    (stroke (width 0) (type default))
-  )
