File: electronics/cube-batteryboard/cube-batteryboard.kicad_pcb (KiCad board)
At the start: 2 copper layers, 95 x 95 mm, 13 parts, among them J1 Conn_01x02, J2 Conn_01x02, SW1 SW_DPST, SW2 SW_DPST

Commit message: Fix unconnected GND circuit for J2 (pin 1)
Connections:
- J2 pad 1: unconnected-(J2-Pin_1-Pad1) -> GND
Changed lines of the file:
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@@
   (net 2 "/PWR_IN")
   (net 3 "/PWR_OUT")
-  (net 4 "unconnected-(J2-Pin_1-Pad1)")
   (footprint "MountingHole:MountingHole_3.2mm_M3_DIN965_Pad" (layer "F.Cu")
     (at 110 25)
@@
       (stroke (width 0.12) (type solid)) (layer "B.Fab"))
     (pad "1" thru_hole roundrect (at 0 0 90) (size 6 6) (drill 4.5) (layers "*.Cu" "*.Mask") (roundrect_rratio 0.25)
-      (net 4 "unconnected-(J2-Pin_1-Pad1)") (pinfunction "Pin_1") (pintype "passive") (thermal_bridge_width 2))
+      (net 1 "GND") (pinfunction "Pin_1") (pintype "passive") (thermal_bridge_width 2))
     (pad "2" thru_hole circle (at 7.2 0 90) (size 6 6) (drill 4.5) (layers "*.Cu" "*.Mask")
       (net 3 "/PWR_OUT") (pinfunction "Pin_2") (pintype "passive") (thermal_bridge_width 2))

Commit message: fix labels for on off switch
Parts:
- moved kibuzzard-656351D2 25.5 mm to (80.2, 32.0)
- moved kibuzzard-656351E7 25.5 mm to (54.8, 32.0)
Changed lines of the file:
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@@
   )
   (footprint "kibuzzard-656351D2" (layer "B.Cu")
-    (at 54.75 32 90)
+    (at 80.25 32 90)
     (descr "Generated with KiBuzzard")
     (tags "kb_params=eyJBbGlnbm1lbnRDaG9pY2UiOiAiQ2VudGVyIiwgIkNhcExlZnRDaG9pY2UiOiAiKCIsICJDYXBSaWdodENob2ljZSI6ICIpIiwgIkZvbnRDb21ib0JveCI6ICJVYnVudHVNb25vLUIiLCAiSGVpZ2h0Q3RybCI6ICIzIiwgIkxheWVyQ29tYm9Cb3giOiAiRi5TaWxrUyIsICJNdWx0aUxpbmVUZXh0IjogIk9GRiIsICJQYWRkaW5nQm90dG9tQ3RybCI6ICI1IiwgIlBhZGRpbmdMZWZ0Q3RybCI6ICI1IiwgIlBhZGRpbmdSaWdodEN0cmwiOiAiNSIsICJQYWRkaW5nVG9wQ3RybCI6ICI1IiwgIldpZHRoQ3RybCI6ICIifQ==")
@@
   )
   (footprint "kibuzzard-656351E7" (layer "B.Cu")
-    (at 80.25 32 90)
+    (at 54.75 32 90)
     (descr "Generated with KiBuzzard")
     (tags "kb_params=eyJBbGlnbm1lbnRDaG9pY2UiOiAiQ2VudGVyIiwgIkNhcExlZnRDaG9pY2UiOiAiKCIsICJDYXBSaWdodENob2ljZSI6ICIpIiwgIkZvbnRDb21ib0JveCI6ICJVYnVudHVNb25vLUIiLCAiSGVpZ2h0Q3RybCI6ICIzIiwgIkxheWVyQ29tYm9Cb3giOiAiRi5TaWxrUyIsICJNdWx0aUxpbmVUZXh0IjogIk9OIiwgIlBhZGRpbmdCb3R0b21DdHJsIjogIjUiLCAiUGFkZGluZ0xlZnRDdHJsIjogIjUiLCAiUGFkZGluZ1JpZ2h0Q3RybCI6ICI1IiwgIlBhZGRpbmdUb3BDdHJsIjogIjUiLCAiV2lkdGhDdHJsIjogIiJ9")
